File: GamePad_I2S_audio_Buttons/KiCad/GamePad_I2S_audio.kicad_pcb (KiCad board)
At the start: 4 copper layers, 47.1 x 33.5 mm, 84 parts, among them IC1 PCM5100, IC2 PAM8908, IC3 TLV61225DC, J1 Conn_02x17_Odd_Even

Commit message: Better GND
Routing:
- net GNDA: track 122.2 -> 143.4 mm, vias 12 -> 27
- net /+3V3: track 59.8 -> 43.7 mm
- net +3V3A: track 52.1 -> 45.8 mm
- net Net-(LED1-K): track 12.2 -> 11.2 mm
- net /WC_B3: track 9.87 -> 10.4 mm
- net GND: track 33.7 -> 33.8 mm, vias 32 -> 50

Commit message: Update
Parts:
- added H1: MountingHole, MountingHole:MountingHole_2mm, F.Cu at (135.2, 84.8)
- moved LED0 11.6 mm to (156.0, 84.9)
- moved LED7 11.3 mm to (156.0, 73.7)
- moved LED1 8.56 mm to (156.0, 83.3)
- moved LED6 8.26 mm to (156.0, 75.3)
- moved LED2 5.59 mm to (156.0, 81.7)
- moved LED5 5.32 mm to (156.0, 76.9)
- moved LED3 3.15 mm to (156.0, 80.1)
- moved LED4 2.98 mm to (156.0, 78.5)
- moved CAP1 1.93 mm to (145.8, 66.3)
- moved CAP2 0.94 mm to (121.5, 66.3)
- moved REF** 0.87 mm to (154.8, 57.5)
Connections:
- C11 pad 2: GNDA -> GND
- C12 pad 2: GNDA -> GND
- C14 pad 2: GNDA -> GND
- C18 pad 2: GNDA -> GND
- C19 pad 2: GNDA -> GND
- C5 pad 2: GNDA -> GND
- C6 pad 2: GNDA -> GND
- C8 pad 1: GNDA -> GND
- C9 pad 2: GNDA -> GND
- IC1 pad 3: GNDA -> GND
- IC1 pad 9: GNDA -> GND
- R0 pad 1: Net-(LED0-K) -> Net-(LED7-K)
- R1 pad 1: Net-(LED1-K) -> Net-(LED6-K)
- R2 pad 1: Net-(LED2-K) -> Net-(LED5-K)
- R21 pad 2: GNDA -> GND
- R3 pad 1: Net-(LED3-K) -> Net-(LED4-K)
- R4 pad 1: Net-(LED4-K) -> Net-(LED3-K)
- R5 pad 1: Net-(LED5-K) -> Net-(LED2-K)
- R6 pad 1: Net-(LED6-K) -> Net-(LED1-K)
- R7 pad 1: Net-(LED7-K) -> Net-(LED0-K)
Routing:
- net GNDA: track 143.4 -> 0.00 mm, vias 27 -> 0
- net GND: track 33.8 -> 175.3 mm, vias 50 -> 76
- net Net-(LED0-K): track 9.34 -> 23.9 mm
- net Net-(LED1-K): track 11.2 -> 22.2 mm
- net Net-(LED7-K): track 22.3 -> 12.0 mm
- net Net-(LED2-K): track 12.7 -> 20.6 mm
- net Net-(LED6-K): track 20.0 -> 13.9 mm
- net Net-(LED3-K): track 14.4 -> 18.9 mm
- net Net-(LED5-K): track 17.9 -> 15.4 mm
- net +1V8: track 20.8 -> 23.2 mm
- net Net-(LED4-K): track 16.2 -> 17.1 mm
- added copper zone on F.Cu, net GND
- removed copper zone on B.Cu, net GNDA
- removed copper zone on F.Cu, net GNDA

Commit message: V1.0
Other:
- board text added: "For Blender export all parts need to be WRL"
- board text added: "PCB_BR_GamePad with I2S Audio v1.0"
- board text added: "PCB_TL_GamePad with I2S Audio v1.0"
Changed lines of the file:
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@@
 		(legacy_teardrops no)
 	)
-	(paper "A4")
+	(paper "A5")
 	(title_block
-		(date "2024-07-18")
+		(title "GamePad I2S Audio")
+		(date "2024-10-18")
+		(rev "v1.0")
 		(company "Intergalaktik d.o.o.")
+		(comment 1 "CERN-OHL-S v2")
 	)
 	(layers
@@
 		(tags "LED")
 		(property "Reference" "LED7"
-			(at -3.141667 0.090001 360)
+			(at -3.141667 0.090001 0)
 			(layer "F.SilkS")
 			(effects
@@
 		)
 		(property "Value" "LED"
-			(at 0 1.43 360)
+			(at 0 1.43 0)
 			(layer "F.Fab")
 			(hide yes)
@@
 		)
 		(fp_text user "${REFERENCE}"
-			(at 0 0 360)
+			(at 0 0 0)
 			(layer "F.Fab")
 			(effects
@@
 		(tags "LED")
 		(property "Reference" "LED0"
-			(at -3.141667 -0.119999 360)
+			(at -3.141667 -0.119999 0)
 			(layer "F.SilkS")
 			(effects
@@
 		)
 		(property "Value" "LED"
-			(at 0 1.43 360)
+			(at 0 1.43 0)
 			(layer "F.Fab")
 			(hide yes)
@@
 		)
 		(fp_text user "${REFERENCE}"
-			(at 0 0 360)
+			(at 0 0 0)
 			(layer "F.Fab")
 			(effects
@@
 		(tags "LED")
 		(property "Reference" "LED2"
-			(at -3.141667 -0.009999 360)
+			(at -3.141667 -0.009999 0)
 			(layer "F.SilkS")
 			(effects
@@
 		)
 		(property "Value" "LED"
-			(at 0 1.43 360)
+			(at 0 1.43 0)
 			(layer "F.Fab")
 			(hide yes)
@@
 		(tags "LED")
 		(property "Reference" "LED3"
-			(at -3.141667 -0.109999 360)
+			(at -3.141667 -0.109999 0)
 			(layer "F.SilkS")
 			(effects
@@
 		)
 		(property "Value" "LED"
-			(at 0 1.43 360)
+			(at 0 1.43 0)
 			(layer "F.Fab")
 			(hide yes)
@@
 		)
 		(fp_text user "${REFERENCE}"
-			(at 0 0 360)
+			(at 0 0 0)
 			(layer "F.Fab")
 			(effects
@@
 		(tags "LED")
 		(property "Reference" "LED6"
-			(at -3.141667 -0.109999 360)
+			(at -3.141667 -0.109999 0)
 			(layer "F.SilkS")
 			(effects
@@
 		)
 		(property "Value" "LED"
-			(at 0 1.43 360)
+			(at 0 1.43 0)
 			(layer "F.Fab")
 			(hide yes)
@@
 		)
 		(fp_text user "${REFERENCE}"
-			(at 0 0 360)
+			(at 0 0 0)
 			(layer "F.Fab")
 			(effects
@@
 		(tags "LED")
 		(property "Reference" "LED1"
-			(at -3.141667 -0.009999 360)
+			(at -3.141667 -0.009999 0)
 			(layer "F.SilkS")
 			(effects
@@
 		)
 		(property "Value" "LED"
-			(at 0 1.43 360)
+			(at 0 1.43 0)
 			(layer "F.Fab")
 			(hide yes)
@@
 		)
 		(fp_text user "${REFERENCE}"
-			(at 0 0 360)
+			(at 0 0 0)
 			(layer "F.Fab")
 			(effects
@@
 		(tags "LED")
 		(property "Reference" "LED5"
-			(at -3.141667 -0.009999 360)
+			(at -3.141667 -0.009999 0)
 			(layer "F.SilkS")
 			(effects
@@
 		)
 		(property "Value" "LED"
-			(at 0 1.43 360)
+			(at 0 1.43 0)
 			(layer "F.Fab")
 			(hide yes)
@@
 		)
 		(fp_text user "${REFERENCE}"
-			(at 0 0 360)
+			(at 0 0 0)
 			(layer "F.Fab")
 			(effects
@@
 		(tags "LED")
 		(property "Reference" "LED4"
-			(at -3.141667 -0.009999 360)
+			(at -3.141667 -0.009999 0)
 			(layer "F.SilkS")
 			(effects
@@
 		)
 		(property "Value" "LED"
-			(at 0 1.43 360)
+			(at 0 1.43 0)
 			(layer "F.Fab")
 			(hide yes)
@@
 		)
 		(fp_text user "${REFERENCE}"
-			(at 0 0 360)
+			(at 0 0 0)
 			(layer "F.Fab")
 			(effects
@@
 		)
 	)
+	(gr_text "PCB_TL_GamePad with I2S Audio v1.0"
+		(at 111.29 53.55 0)
+		(layer "Dwgs.User")
+		(effects
+			(font
+				(size 1 1)
+				(thickness 0.15)
+			)
+			(justify left bottom)
+		)
+	)
+	(gr_text "PCB_BR_GamePad with I2S Audio v1.0"
+		(at 158.59 87.17 0)
+		(layer "Dwgs.User")
+		(effects
+			(font
+				(size 1 1)
+				(thickness 0.15)
+			)
+			(justify left bottom)
+		)
+	)
+	(gr_text "For Blender export all parts need to be WRL"
+		(at 111.42 50.76 0)
+		(layer "Dwgs.User")
+		(effects
+			(font
+				(size 1 1)
+				(thickness 0.15)
+			)
+			(justify left bottom)
+		)
+	)
+	(dimension
+		(type aligned)
+		(layer "Cmts.User")
+		(pts
+			(xy 112.433562 53.610634) (xy 112.420634 87.136388)
+		)
+		(height 3.747363)
+		(gr_text "33.5258 mm"
+			(at 107.529735 70.371623 89.97790595)
+			(layer "Cmts.User")
+			(effects
+				(font
+					(size 1 1)
+					(thickness 0.15)
+				)
+			)
+		)
+		(format
+			(prefix "")
+			(suffix "")
+			(units 3)
+			(units_format 1)
+			(precision 4)
+		)
+		(style
+			(thickness 0.1)
+			(arrow_length 1.27)
+			(text_position_mode 0)
+			(extension_height 0.58642)
+			(extension_offset 0.5) keep_text_aligned)
+	)
+	(dimension
+		(type aligned)
+		(layer "Cmts.User")
+		(pts
+			(xy 111.430634 86.136438) (xy 158.526388 86.149366)
+		)
+		(height 4.855568)
+		(gr_text "47.0958 mm"
+			(at 134.977494 89.84847 359.984272)
+			(layer "Cmts.User")
+			(effects
+				(font
+					(size 1 1)
+					(thickness 0.15)
+				)
+			)
+		)
+		(format
+			(prefix "")
+			(suffix "")
+			(units 3)
+			(units_format 1)
+			(precision 4)
+		)
+		(style
+			(thickness 0.1)
+			(arrow_length 1.27)
+			(text_position_mode 0)
+			(extension_height 0.58642)
+			(extension_offset 0.5) keep_text_aligned)
+	)
 	(segment
