File: GamePad_I2S_audio_Buttons/KiCad/GamePad_I2S_audio.kicad_pcb (KiCad board)
At the start: 4 copper layers, 47.1 x 33.5 mm, 85 parts, among them IC1 PCM5100, IC2 PAM8908, IC3 TLV61225DC, J1 Conn_02x17_Odd_Even

Commit message: fix #1
Connections:
- BTN5 pad 1: Net-(BTN5-Pad1) -> (no net)
- BTN5 pad 3: (no net) -> Net-(BTN5-1)
- C26 pad 1: Net-(BTN5-Pad1) -> Net-(BTN5-1)
- R17 pad 2: Net-(BTN5-Pad1) -> Net-(BTN5-1)
- R19 pad 1: Net-(BTN5-Pad1) -> Net-(BTN5-1)
Routing:
- net Net-(BTN5-Pad1): track 20.5 -> 0.00 mm, vias 1 -> 0
- net Net-(BTN5-1): track 0.00 -> 17.5 mm, vias 0 -> 1
Changed lines of the file:
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@@
 	(net 13 "/SER_TX_N")
 	(net 14 "/WB_A8")
-	(net 15 "Net-(BTN5-Pad1)")
+	(net 15 "Net-(BTN5-1)")
 	(net 16 "/EA_A8")
 	(net 17 "/SER_CLK_N")
@@
 			(size 2.3 2.4)
 			(layers "F.Cu" "F.Paste" "F.Mask")
-			(net 15 "Net-(BTN5-Pad1)")
-			(pinfunction "1")
-			(pintype "passive")
 		)
 		(pad "2" smd rect
@@
 			(size 2.3 2.4)
 			(layers "F.Cu" "F.Paste" "F.Mask")
+			(net 15 "Net-(BTN5-1)")
+			(pinfunction "1")
+			(pintype "passive")
 		)
 		(pad "4" smd rect
@@
 			(layers "B.Cu" "B.Paste" "B.Mask")
 			(roundrect_rratio 0.25)
-			(net 15 "Net-(BTN5-Pad1)")
+			(net 15 "Net-(BTN5-1)")
 			(pintype "passive")
 		)
@@
 			(layers "B.Cu" "B.Paste" "B.Mask")
 			(roundrect_rratio 0.25)
-			(net 15 "Net-(BTN5-Pad1)")
+			(net 15 "Net-(BTN5-1)")
 			(pintype "passive")
 		)
@@
 			(layers "B.Cu" "B.Paste" "B.Mask")
 			(roundrect_rratio 0.25)
-			(net 15 "Net-(BTN5-Pad1)")
+			(net 15 "Net-(BTN5-1)")
 			(pintype "passive")
 		)
@@
 	)
 	(gr_text "PCB_BR_GamePad with I2S Audio v1.0"
-		(at 158.59 87.17 0)
+		(at 158.59 87.17 180)
 		(layer "Dwgs.User")
 		(effects
@@
 	)
 	(segment
-		(start 119.93 56.25)
-		(end 120.36 55.82)
-		(width 0.2)
-		(layer "F.Cu")
-		(net 15)
-	)
-	(segment
-		(start 119.93 57.97)
-		(end 119.93 56.25)
-		(width 0.2)
-		(layer "F.Cu")
-		(net 15)
-	)
-	(segment
-		(start 120.36 55.82)
-		(end 120.66 55.52)
+		(start 128.69 63.84)
+		(end 125.18 63.84)
 		(width 0.2)
 		(layer "F.Cu")
@@
 	)
 	(segment
-		(start 120.66 55.52)
-		(end 120.66 54.83)
-		(width 0.2)
-		(layer "F.Cu")
-		(net 15)
-	)
-	(segment
-		(start 128.69 67.35)
-		(end 122.62 61.28)
+		(start 125.18 63.84)
+		(end 119.93 58.59)
 		(width 0.2)
 		(layer "F.Cu")
@@
 	)
 	(segment
-		(start 122.62 61.28)
-		(end 119.93 58.59)
+		(start 119.93 58.59)
+		(end 119.93 56.25)
 		(width 0.2)
 		(layer "F.Cu")
@@
 	)
 	(segment
-		(start 119.93 58.59)
-		(end 119.93 57.97)
+		(start 119.93 56.25)
+		(end 120.66 55.52)
 		(width 0.2)
 		(layer "F.Cu")
@@
 	)
 	(segment
-		(start 128.69 68.84)
-		(end 128.69 67.35)
+		(start 120.66 55.52)
+		(end 120.66 54.83)
 		(width 0.2)
 		(layer "F.Cu")
