File: GamePad_I2S_audio_Buttons/KiCad/GamePad_I2S_audio.kicad_sch (KiCad schematic)
At the start: 79 parts, among them IC1 PCM5100, IC2 PAM8908, IC3 TLV61225DC, J1 Conn_02x17_Odd_Even

Commit message: Update
Parts:
- added H1: MountingHole, MountingHole:MountingHole_2mm, symbol Mechanical:MountingHole
Connections:
- net GNDA is gone; now on net GND: C11.2, C12.2, C14.2, C18.2, C19.2, C5.2, C6.2, C8.1, C9.2, IC1.3 (CPGND), IC1.9 (AGND), R21.2
- net at R3.1: now also LED4.1 (K); no longer LED3.1 (K)
- net at LED7.1 (K): now also R0.1; no longer R7.1
- net at LED0.1 (K): now also R7.1; no longer R0.1
- net at R1.1: now also LED6.1 (K); no longer LED1.1 (K)
- net at R4.1: now also LED3.1 (K); no longer LED4.1 (K)
- net at LED2.1 (K): now also R5.1; no longer R2.1
- net at LED5.1 (K): now also R2.1; no longer R5.1
- net at R6.1: now also LED1.1 (K); no longer LED6.1 (K)
Other:
- moved on the sheet: LED0, LED1, LED2, LED3, LED4, LED5, LED6, LED7
Changed lines of the file:
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@@
 	(symbol
 		(lib_id "Device:LED")
-		(at 92.71 66.04 180)
+		(at 92.71 30.48 180)
 		(unit 1)
 		(exclude_from_sim no)
@@
 		(dnp no)
 		(property "Reference" "LED7"
-			(at 88.646 67.31 0)
+			(at 88.646 31.75 0)
 			(effects
 				(font
@@
 		)
 		(property "Value" "LED"
-			(at 96.012 67.31 0)
+			(at 96.012 31.75 0)
 			(effects
 				(font
@@
 		)
 		(property "Footprint" "LED_SMD:LED_0603_1608Metric"
-			(at 92.71 66.04 0)
+			(at 92.71 30.48 0)
 			(effects
 				(font
@@
 		)
 		(property "Datasheet" "~"
-			(at 92.71 66.04 0)
+			(at 92.71 30.48 0)
 			(effects
 				(font
@@
 		)
 		(property "Description" "Light emitting diode"
-			(at 92.71 66.04 0)
+			(at 92.71 30.48 0)
 			(effects
 				(font
@@
 			)
 		)
-		(property "Value" "GNDA"
+		(property "Value" "GND"
 			(at 191.897 118.6942 0)
 			(effects
@@
 	(symbol
 		(lib_id "Device:LED")
-		(at 92.71 30.48 180)
+		(at 92.71 66.04 180)
 		(unit 1)
 		(exclude_from_sim no)
@@
 		(dnp no)
 		(property "Reference" "LED0"
-			(at 88.392 32.004 0)
+			(at 88.392 67.564 0)
 			(effects
 				(font
@@
 		)
 		(property "Value" "LED"
-			(at 96.012 31.75 0)
+			(at 96.012 67.31 0)
 			(effects
 				(font
@@
 		)
 		(property "Footprint" "LED_SMD:LED_0603_1608Metric"
-			(at 92.71 30.48 0)
+			(at 92.71 66.04 0)
 			(effects
 				(font
@@
 		)
 		(property "Datasheet" "~"
-			(at 92.71 30.48 0)
+			(at 92.71 66.04 0)
 			(effects
 				(font
@@
 		)
 		(property "Description" "Light emitting diode"
-			(at 92.71 30.48 0)
+			(at 92.71 66.04 0)
 			(effects
 				(font
@@
 			)
 		)
-		(property "Value" "GNDA"
+		(property "Value" "GND"
 			(at 232.9942 54.737 90)
 			(effects
@@
 			)
 		)
-		(property "Value" "GNDA"
+		(property "Value" "GND"
 			(at 212.6742 54.737 90)
 			(effects
@@
 			)
 		)
-		(property "Value" "GNDA"
+		(property "Value" "GND"
 			(at 132.6642 58.547 90)
 			(effects
@@
 	(symbol
 		(lib_id "Device:LED")
-		(at 92.71 50.8 180)
+		(at 92.71 45.72 180)
 		(unit 1)
 		(exclude_from_sim no)
@@
 		(dnp no)
 		(property "Reference" "LED4"
-			(at 88.646 52.07 0)
+			(at 88.646 46.99 0)
 			(effects
 				(font
@@
 		)
 		(property "Value" "LED"
-			(at 96.012 52.07 0)
+			(at 96.012 46.99 0)
 			(effects
 				(font
@@
 		)
 		(property "Footprint" "LED_SMD:LED_0603_1608Metric"
-			(at 92.71 50.8 0)
+			(at 92.71 45.72 0)
 			(effects
 				(font
@@
 		)
 		(property "Datasheet" "~"
-			(at 92.71 50.8 0)
+			(at 92.71 45.72 0)
 			(effects
 				(font
@@
 		)
 		(property "Description" "Light emitting diode"
-			(at 92.71 50.8 0)
+			(at 92.71 45.72 0)
 			(effects
 				(font
@@
 	(symbol
 		(lib_id "Device:LED")
-		(at 92.71 40.64 180)
+		(at 92.71 55.88 180)
 		(unit 1)
 		(exclude_from_sim no)
@@
 		(dnp no)
 		(property "Reference" "LED2"
-			(at 88.646 41.91 0)
+			(at 88.646 57.15 0)
 			(effects
 				(font
@@
 		)
 		(property "Value" "LED"
-			(at 96.012 41.91 0)
+			(at 96.012 57.15 0)
 			(effects
 				(font
@@
 		)
 		(property "Footprint" "LED_SMD:LED_0603_1608Metric"
-			(at 92.71 40.64 0)
+			(at 92.71 55.88 0)
 			(effects
 				(font
@@
 		)
 		(property "Datasheet" "~"
-			(at 92.71 40.64 0)
+			(at 92.71 55.88 0)
 			(effects
 				(font
@@
 		)
 		(property "Description" "Light emitting diode"
-			(at 92.71 40.64 0)
+			(at 92.71 55.88 0)
 			(effects
 				(font
@@
 	(symbol
 		(lib_id "Device:LED")
-		(at 92.71 60.96 180)
+		(at 92.71 35.56 180)
 		(unit 1)
 		(exclude_from_sim no)
@@
 		(dnp no)
 		(property "Reference" "LED6"
-			(at 88.646 62.23 0)
+			(at 88.646 36.83 0)
 			(effects
 				(font
@@
 		)
 		(property "Value" "LED"
-			(at 96.012 62.23 0)
+			(at 96.012 36.83 0)
 			(effects
 				(font
@@
 		)
 		(property "Footprint" "LED_SMD:LED_0603_1608Metric"
-			(at 92.71 60.96 0)
+			(at 92.71 35.56 0)
 			(effects
 				(font
@@
 		)
 		(property "Datasheet" "~"
-			(at 92.71 60.96 0)
+			(at 92.71 35.56 0)
 			(effects
 				(font
@@
 		)
 		(property "Description" "Light emitting diode"
-			(at 92.71 60.96 0)
+			(at 92.71 35.56 0)
 			(effects
 				(font
@@
 			)
 		)
-		(property "Value" "GNDA"
+		(property "Value" "GND"
 			(at 166.497 141.5542 0)
 			(effects
@@
 	(symbol
 		(lib_id "Device:LED")
-		(at 92.71 55.88 180)
+		(at 92.71 40.64 180)
 		(unit 1)
 		(exclude_from_sim no)
@@
 		(dnp no)
 		(property "Reference" "LED5"
-			(at 88.646 57.15 0)
+			(at 88.646 41.91 0)
 			(effects
 				(font
@@
 		)
 		(property "Value" "LED"
-			(at 96.012 57.15 0)
+			(at 96.012 41.91 0)
 			(effects
 				(font
@@
 		)
 		(property "Footprint" "LED_SMD:LED_0603_1608Metric"
-			(at 92.71 55.88 0)
+			(at 92.71 40.64 0)
 			(effects
 				(font
@@
 		)
 		(property "Datasheet" "~"
-			(at 92.71 55.88 0)
+			(at 92.71 40.64 0)
 			(effects
 				(font
@@
 		)
 		(property "Description" "Light emitting diode"
-			(at 92.71 55.88 0)
+			(at 92.71 40.64 0)
 			(effects
 				(font
@@
 	(symbol
 		(lib_id "Device:LED")
-		(at 92.71 35.56 180)
+		(at 92.71 60.96 180)
 		(unit 1)
 		(exclude_from_sim no)
@@
 		(dnp no)
 		(property "Reference" "LED1"
-			(at 88.646 36.83 0)
+			(at 88.646 62.23 0)
 			(effects
 				(font
@@
 		)
 		(property "Value" "LED"
-			(at 96.012 36.83 0)
+			(at 96.012 62.23 0)
 			(effects
 				(font
@@
 		)
 		(property "Footprint" "LED_SMD:LED_0603_1608Metric"
-			(at 92.71 35.56 0)
+			(at 92.71 60.96 0)
 			(effects
 				(font
@@
 		)
 		(property "Datasheet" "~"
-			(at 92.71 35.56 0)
+			(at 92.71 60.96 0)
 			(effects
 				(font
@@
 		)
 		(property "Description" "Light emitting diode"
-			(at 92.71 35.56 0)
+			(at 92.71 60.96 0)
 			(effects
 				(font
@@
 	)
 	(symbol
+		(lib_id "Mechanical:MountingHole")
+		(at 248.92 161.29 0)
+		(unit 1)
+		(exclude_from_sim yes)
+		(in_bom no)
+		(on_board yes)
+		(dnp no)
+		(fields_autoplaced yes)
+		(property "Reference" "H1"
+			(at 251.46 160.0199 0)
+			(effects
+				(font
+					(size 1.27 1.27)
+				)
+				(justify left)
+			)
+		)
+		(property "Value" "MountingHole"
+			(at 251.46 162.5599 0)
+			(effects
+				(font
+					(size 1.27 1.27)
+				)
+				(justify left)
+			)
+		)
+		(property "Footprint" "MountingHole:MountingHole_2mm"
+			(at 248.92 161.29 0)
+			(effects
+				(font
+					(size 1.27 1.27)
+				)
+				(hide yes)
+			)
+		)
+		(property "Datasheet" "~"
+			(at 248.92 161.29 0)
+			(effects
+				(font
+					(size 1.27 1.27)
+				)
+				(hide yes)
+			)
+		)
+		(property "Description" "Mounting Hole without connection"
+			(at 248.92 161.29 0)
+			(effects
+				(font
+					(size 1.27 1.27)
+				)
+				(hide yes)
+			)
+		)
+		(instances
+			(project ""
+				(path "/0dd9b205-0a74-496f-82ec-852763bdf394"
+					(reference "H1")
+					(unit 1)
+				)
+			)
+		)
+	)
+	(symbol
 		(lib_id "OLIMEX_Power:+1V8")
 		(at 85.09 55.88 90)
@@
 	(symbol
 		(lib_id "Device:LED")
-		(at 92.71 45.72 180)
+		(at 92.71 50.8 180)
 		(unit 1)
 		(exclude_from_sim no)
@@
 		(dnp no)
 		(property "Reference" "LED3"
-			(at 88.646 46.99 0)
+			(at 88.646 52.07 0)
 			(effects
 				(font
@@
 		)
 		(property "Value" "LED"
-			(at 96.012 46.99 0)
+			(at 96.012 52.07 0)
 			(effects
 				(font
@@
 		)
 		(property "Footprint" "LED_SMD:LED_0603_1608Metric"
-			(at 92.71 45.72 0)
+			(at 92.71 50.8 0)
 			(effects
 				(font
@@
 		)
 		(property "Datasheet" "~"
-			(at 92.71 45.72 0)
+			(at 92.71 50.8 0)
 			(effects
 				(font
@@
 		)
 		(property "Description" "Light emitting diode"
-			(at 92.71 45.72 0)
+			(at 92.71 50.8 0)
 			(effects
 				(font

Commit message: fix #1
Connections:
- net at C26.1, R17.2, R19.1: now also BTN5.3 (1); no longer BTN5.1
Changed lines of the file:
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@@
 	)
 	(symbol
+		(lib_name "SW_Push_1")
 		(lib_id "Switch:SW_Push")
 		(at 48.26 182.88 0)
@@
 			)
 		)
-		(pin "1"
+		(pin "3"
 		)
 		(pin "2"
