File: extension_template/extension_template.kicad_sch (KiCad schematic)
At the start: 17 parts, among them J6 MISC

Commit message: Template update
Parts:
- FID1: value Fiducial -> Fiducial_F_TL
- FID2: value Fiducial -> Fiducial_F_TR
- FID3: value Fiducial -> Fiducial_F_BL
- FID4: value Fiducial -> Fiducial_B_TL
- FID5: value Fiducial -> Fiducial_B_TR
- FID6: value Fiducial -> Fiducial_B_BL
Connections:
- net Power/2V5 is gone; now on net +2V5: F1.2
- net +2V5: no longer F1.1, J6.1 (Pin_1)
- new net +Exten_V: F1.1, J6.1 (Pin_1)
Other:
- note added: "!!!!!!!!!!!!!!!!!!!!!!!!!!!!!!!!!!!!!!!!! There is same pinout part for 5V step up. So you can have 5V with just one IC change. For more details check Power page. !!!!!!!!!!!!!!!!!!!!!!!!!!!!!!!!!!!!!!!!!"
- note added: "!!!!!!!!!!!!!!!!!!!!!!!!!!!!!!!!!!!!!!!!!!!!!!!!! Olimex board is delivering MAX 2.5V on connector. You can use 2.5V output signals for 3.3V. Be carefull FPGA input only tolerate MAX 2.5V! !!!!!!!!!!!!!!!!!!!!!!!!!!!!!!!!!!!!!!!!!!!!!!!!!"
- note added: "!!!!!!!!!!!!!!!!!!!!!!!!!!!!!!!!!!!!!!!!!!!!!!!!!!!!!!!!!!!!! 2.5V input is connected over 500mA resetable fuse! Maximum current for 2.5V is set to 500mA. It may be possible to drain more current but you will need add different FUSE and use it at your own risk! 3.3V step up is limited to 300mA Idea behind limits is that you can use all 3 extensions slots at once without any risk od draining to mu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"
- note added: "${project_name} ${project_version}"
- note added: "Bottom View"
- note added: "Change project informations under. File>>Schamatic Setup>>Text Variables"
- note added: "Dimensions"
- note added: "Fiducials"
- note added: "Replace bottom 3D images with your PCB"
- note added: "TEST points"
- note added: "Top View"
- company: Intergalaktik d.o.o. -> ${project_creator}
- title: olimex extension template -> ${project_name} ${project_version}
- moved on the sheet: F1, FID1, FID2, FID3, FID4, FID5, FID6, H1, H2, H3, H4, H5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

Commit message: Extension template update
Parts:
- removed F1: 0805L050WR, Fuse:Fuse_0805_2012Metric, symbol Device:Fuse_Small
- removed FID1: Fiducial_F_TL, Fiducial:Fiducial_0.5mm_Mask1mm, symbol Mechanical:Fiducial
- removed FID2: Fiducial_F_TR, Fiducial:Fiducial_0.5mm_Mask1mm, symbol Mechanical:Fiducial
- removed FID3: Fiducial_F_BL, Fiducial:Fiducial_0.5mm_Mask1mm, symbol Mechanical:Fiducial
- removed FID4: Fiducial_B_TL, Fiducial:Fiducial_0.5mm_Mask1mm, symbol Mechanical:Fiducial
- removed FID5: Fiducial_B_TR, Fiducial:Fiducial_0.5mm_Mask1mm, symbol Mechanical:Fiducial
- removed FID6: Fiducial_B_BL, Fiducial:Fiducial_0.5mm_Mask1mm, symbol Mechanical:Fiducial
- removed H1: Logo Intergalaktik, intergalaktik:intergalaktik, symbol Mechanical:MountingHole
- removed H2: Logo NLnet, nlnet:nlnet, symbol Mechanical:MountingHole
- removed H3: Logo OpenCologne, Cologne:open_cologne_small, symbol Mechanical:MountingHole
- removed H4: Logo Radiona, radiona:radiona_small, symbol Mechanical:MountingHole
- removed H5, H6: MountingHole, MountingHole:MountingHole_2.2mm_M2, symbol Mechanical:MountingHole
- removed J6: MISC, Connector_PinSocket_2.54mm:PinSocket_2x10_P2.54mm_Vertical_SMD, symbol Connector_Generic:Conn_02x10_Odd_Even
- removed TP1: 3V3, TestPoint:TestPoint_Pad_D1.0mm, symbol Connector:TestPoint_Probe
- removed TP2: 2V5, TestPoint:TestPoint_Pad_D1.0mm, symbol Connector:TestPoint_Probe
- removed TP3: GND, TestPoint:TestPoint_Pad_D1.0mm, symbol Connector:TestPoint_Probe
Other:
- removed sheet Power
- added sheet Main Sheet (main.kicad_sch)
- note added: "......"
- note added: "......."
- note added: "1"
- note added: "2"
- note added: "3"
- note added: "BOTTOM VIEW"
- note added: "CoverPage"
- note added: "DIMENSIONS"
- note added: "Index"
- note added: "MainPage"
- note added: "Page"
- note added: "PowerPage"
- note added: "TOP VIEW"
- note removed: "2V5 over Resettable Fuses - PPTC 0.50A 6V 0805 >3V3"
- note removed: "Bottom View"
- note removed: "Dimensions"
- note removed: "Fiducials"
- note removed: "OLIMEX CONNECTOR"
- note removed: "POWER FLAGS"
- note removed: "TEST points"
- note removed: "Top View"

Commit message: Template update
Other:
- added sheet Dimension (dimension.kicad_sch)
- note added: "4"
- note added: "Board Dimensions"
- note removed: "DIMENSIONS"
