File: extension_template/extension_template.kicad_sch (KiCad schematic)
At the start: 0 parts

Commit message: Adding git ignore
Other:
- note added: "${CURRENT_DATE}"
Changed lines of the file:
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@@
 		)
 	)
-	(text_box "Project creator: ${project_creator}\nProject License: ${project_license}\nYear: ${project_year}"
+	(text_box "${project_creator}\nLicense: ${project_license}\nYear: ${project_year}"
 		(exclude_from_sim no)
 		(at 16.51 22.098 0)
@@
 		)
 	)
+	(text "${CURRENT_DATE}"
+		(exclude_from_sim no)
+		(at 257.556 17.526 0)
+		(effects
+			(font
+				(size 5.08 5.08)
+				(thickness 0.762)
+				(bold yes)
+			)
+		)
+	)

Commit message: Template update
Other:
- note added: "!!!!!!!!!!!!!!!!!!!!!!!!!!!!!!!!!!!!!!!!!!!!!!!!!!!!!!!!!!!!! VCC input is connected over 500mA resetable fuse! Maximum current for VCC is set to 500mA. It may be possible to drain more current but you will need add different FUSE and use it at your own risk! 3.3V step up is limited to 400mA Idea behind limits is that you can use all 3 extensions slots at once without any risk od draining to much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"
- note added: "A1 Dedicated clock input pins are: IO_SB_A8: CLK0 IO_SB_A7: CLK1 IO_SB_A6: CLK2 IO_SB_A5: CLK3 You can use them all as differential inputs. We are not able to use any on extension boards. It is also possible to use any GPIO as a clock input. The only thing to note here is that the signal must be routed via the routing structure to the entry point of the global clock mesh. These paths are longer t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"
- note removed: "!!!!!!!!!!!!!!!!!!!!!!!!!!!!!!!!!!!!!!!!!!!!!!!!!!!!!!!!!!!!! 2.5V input is connected over 500mA resetable fuse! Maximum current for 2.5V is set to 500mA. It may be possible to drain more current but you will need add different FUSE and use it at your own risk! 3.3V step up is limited to 300mA Idea behind limits is that you can use all 3 extensions slots at once without any risk od draining to mu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"
Changed lines of the file:
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@@
 	)
 	(rectangle
+		(start 227.838 36.83)
+		(end 282.956 68.58)
+		(stroke
+			(width 0.127)
+			(type dash)
+		)
+		(fill
+			(type color)
+			(color 158 196 255 1)
+		)
+	)
+	(rectangle
 		(start 18.034 58.928)
 		(end 120.396 90.424)
@@
 		(fill
 			(type color)
-			(color 255 255 0 1)
+			(color 255 0 0 0.5)
 		)
 	)
@@
 		)
 		(fill
-			(type none)
+			(type color)
+			(color 0 255 0 0.1)
 		)
 	)
@@
 		(fill
 			(type color)
-			(color 255 255 0 1)
+			(color 0 255 0 0.5)
 		)
 	)
@@
 		)
 	)
-	(text "!!!!!!!!!!!!!!!!!!!!!!!!!!!!!!!!!!!!!!!!!!!!!!!!!!!!!!!!!!!!!\n2.5V input is connected over 500mA resetable fuse!\nMaximum current for 2.5V is set to 500mA.\nIt may be possible to drain more current but \nyou will need add different FUSE and use it at your own risk!\n3.3V step up is limited to 300mA \nIdea behind limits is that you can use all 3 extensions slots \nat once without any risk od draining to much!\n!!!!!!!!!!!!!!!!!!!!!!!!!!!!!!!!!!!!!!!!!!!!!!!!!!!!!!!!!!!!!"
+	(text "!!!!!!!!!!!!!!!!!!!!!!!!!!!!!!!!!!!!!!!!!!!!!!!!!!!!!!!!!!!!!\nVCC input is connected over 500mA resetable fuse!\nMaximum current for VCC is set to 500mA.\nIt may be possible to drain more current but \nyou will need add different FUSE and use it at your own risk!\n3.3V step up is limited to 400mA \nIdea behind limits is that you can use all 3 extensions slots \nat once without any risk od draining to much!\n!!!!!!!!!!!!!!!!!!!!!!!!!!!!!!!!!!!!!!!!!!!!!!!!!!!!!!!!!!!!!"
 		(exclude_from_sim no)
 		(at 68.58 75.184 0)
@@
 			(font
 				(size 2.032 2.032)
-				(color 132 0 0 1)
+				(color 0 0 0 1)
 			)
 		)
@@
 			(font
 				(size 2.032 2.032)
-				(color 132 0 0 1)
+				(color 0 0 0 1)
 			)
 		)
@@
 			(font
 				(size 2.032 2.032)
-				(color 132 0 0 1)
+				(color 0 0 0 1)
 			)
 		)
@@
 			)
 		)
+	)
+	(text "A1 Dedicated clock input pins are:\n    IO_SB_A8: CLK0\n    IO_SB_A7: CLK1\n    IO_SB_A6: CLK2\n    IO_SB_A5: CLK3\nYou can use them all as differential inputs.\n\nWe are not able to use any on extension boards.\n\nIt is also possible to use any GPIO as a clock input. \nThe only thing to note here is that the signal must be \nrouted via the routing structure to the entry point \nof the global clock mesh. These paths are longer than \nvia the dedicated clock pins, which is why it is \nessential to pay attention to clock skew."
+		(exclude_from_sim no)
+		(at 256.032 52.832 0)
+		(effects
+			(font
+				(size 1.27 1.27)
+				(color 0 0 0 1)
+			)
+		)
