File: extension_template/extension_template.kicad_pcb (KiCad board)
At the start: 4 copper layers, 30 x 30 mm, 23 parts, among them IC3 TLV61225DC, J6 MISC

Commit message: Template update
Parts:
- moved FID3 10.7 mm to (86.1, 81.0)
- moved FID6 10.7 mm to (114.4, 81.0)
- moved H2 10.7 mm to (90.9, 75.5)
- moved J6 10.7 mm to (100.2, 77.2)
- moved TP1 10.7 mm to (87.1, 72.5)
- moved FID1 10.7 mm to (90.8, 52.8)
- moved FID2 10.7 mm to (109.7, 52.8)
- moved FID4 10.7 mm to (109.7, 52.8)
- moved FID5 10.7 mm to (90.8, 52.8)
- moved TP3 10.7 mm to (87.1, 62.6)
- moved C13 10.7 mm to (90.2, 67.7)
- moved C14 10.7 mm to (92.0, 65.4)
- moved H1 10.7 mm to (95.9, 78.5)
- moved H4 10.7 mm to (99.7, 74.8)
- moved H5 10.7 mm to (88.3, 54.8)
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
Commit message: TEmplate update
Parts:
- FID1: value Fiducial -> Fiducial_F_TL
- FID2: value Fiducial -> Fiducial_F_TR
- FID3: value Fiducial -> Fiducial_F_BL
- FID4: value Fiducial -> Fiducial_B_TL
- FID5: value Fiducial -> Fiducial_B_TR
- FID6: value Fiducial -> Fiducial_B_BL
Connections:
- net /NB_A0 renamed /Main Sheet/NB_A0
- net /NB_A1 renamed /Main Sheet/NB_A1
- net /NB_A2 renamed /Main Sheet/NB_A2
- net /NB_A3 renamed /Main Sheet/NB_A3
- net /NB_A4 renamed /Main Sheet/NB_A4
- net /NB_A5 renamed /Main Sheet/NB_A5
- net /NB_A6 renamed /Main Sheet/NB_A6
- net /NB_A7 renamed /Main Sheet/NB_A7
- net /NB_A8 renamed /Main Sheet/NB_A8
- net /NB_B0 renamed /Main Sheet/NB_B0
- net /NB_B1 renamed /Main Sheet/NB_B1
- net /NB_B2 renamed /Main Sheet/NB_B2
- net /NB_B3 renamed /Main Sheet/NB_B3
- net /NB_B4 renamed /Main Sheet/NB_B4
- net /NB_B5 renamed /Main Sheet/NB_B5
- net /NB_B6 renamed /Main Sheet/NB_B6
- net /NB_B7 renamed /Main Sheet/NB_B7
- net /NB_B8 renamed /Main Sheet/NB_B8
- C13 pad 1: /Power/2V5 -> +2V5
- F1 pad 1: +2V5 -> +Exten_V
- F1 pad 2: /Power/2V5 -> +2V5
- IC3 pad 1: /Power/2V5 -> +2V5
- J6 pad 1: +2V5 -> +Exten_V
- L1 pad 2: /Power/2V5 -> +2V5
- R15 pad 1: /Power/2V5 -> +2V5
Routing:
- net +2V5: track 10.8 -> 23.3 mm
- net /Power/2V5: track 12.5 -> 0.00 mm

Commit message: Template update
Parts:
- moved TP1 12.3 mm to (97.8, 66.5)
- moved H3 1.05 mm to (107.8, 77.6)
Routing:
- net +Exten_V: track 0.00 -> 8.76 mm
- net +2V5: track 23.3 -> 17.7 mm
Changed lines of the file:
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@@
 	(footprint "Cologne:open_cologne_small"
 		(layer "F.Cu")
-		(at 108.82 77.685)
+		(at 107.77 77.64)
 		(property "Reference" "H3"
 			(at 0 0 0)
@@
 	(footprint "TestPoint:TestPoint_Pad_D1.0mm"
 		(layer "F.Cu")
-		(at 87.08 72.5225)
+		(at 97.83 66.46)
 		(descr "SMD pad as test Point, diameter 1.0mm")
 		(tags "test point SMD pad")
@@
 	)
 	(via
-		(at 88.81 72.915)
+		(at 88.82 72.96)
 		(size 0.8)
 		(drill 0.4)
@@
 	)
 	(segment
-		(start 88.82 74.72)
-		(end 88.82 72.925)
-		(width 0.5)
-		(layer "B.Cu")
-		(net 2)
-	)
-	(segment
 		(start 91.67 66.991666)
 		(end 91.67 65.856666)
@@
 	)
 	(segment
-		(start 88.82 72.925)
-		(end 88.81 72.915)
+		(start 88.82 72.96)
+		(end 88.82 74.72)
 		(width 0.5)
 		(layer "B.Cu")
@@
 	)
 	(segment
-		(start 86.15 72.655)
-		(end 86.8075 72.655)
+		(start 96.33 67.96)
+		(end 97.83 66.46)
 		(width 0.5)
 		(layer "F.Cu")
@@
 	)
 	(segment
-		(start 86.8075 72.655)
-		(end 86.94 72.5225)
+		(start 96.33 69.57)
+		(end 96.33 67.96)
 		(width 0.5)
 		(layer "F.Cu")
@@
 	)
 	(via
-		(at 86.15 72.655)
-		(size 0.8)
-		(drill 0.4)
+		(at 96.33 69.57)
+		(size 0.6)
+		(drill 0.3)
 		(layers "F.Cu" "B.Cu")
 		(net 5)
 	)
 	(segment
-		(start 91.7225 69.951666)
-		(end 91.7225 68.344166)
-		(width 0.3)
+		(start 96.311666 69.551666)
+		(end 96.33 69.57)
+		(width 0.5)
 		(layer "B.Cu")
 		(net 5)
 	)
 	(segment
-		(start 86.94 71.78)
-		(end 86.94 71.865)
-		(width 0.5)
+		(start 91.7225 69.951666)
+		(end 91.7225 68.344166)
+		(width 0.3)
 		(layer "B.Cu")
 		(net 5)
@@
 	)
 	(segment
-		(start 86.94 71.865)
-		(end 86.15 72.655)
-		(width 0.5)
+		(start 91.065 68.291666)
+		(end 91.67 68.291666)
+		(width 0.3)
 		(layer "B.Cu")
 		(net 5)
 	)
 	(segment
-		(start 91.065 68.291666)
-		(end 91.67 68.291666)
-		(width 0.3)
+		(start 94.8 69.551666)
+		(end 96.311666 69.551666)
+		(width 0.5)
 		(layer "B.Cu")
 		(net 5)
@@
 	)
 	(segment
-		(start 86.94 76.775)
-		(end 86.94 71.78)
-		(width 0.5)
-		(layer "B.Cu")
-		(net 5)
-	)
-	(segment
 		(start 86.94 69.905)
 		(end 88.806666 69.905)
@@
 	)
 	(segment
-		(start 88.82 79.76)
-		(end 88.82 78.655)
-		(width 0.5)
-		(layer "B.Cu")
-		(net 5)
-	)
-	(segment
-		(start 88.82 78.655)
-		(end 86.94 76.775)
-		(width 0.5)
-		(layer "B.Cu")
-		(net 5)
-	)
-	(segment
 		(start 91.985 71.111666)
 		(end 91.7225 70.849166)
@@
 		(net 5)
 	)
+	(segment
+		(start 86.94 76.775)
+		(end 86.94 71.78)
+		(width 0.5)
+		(layer "B.Cu")
+		(net 6)
+	)
+	(segment
+		(start 88.82 79.76)
+		(end 88.82 78.655)
+		(width 0.5)
+		(layer "B.Cu")
+		(net 6)
+	)
+	(segment
+		(start 88.82 78.655)
+		(end 86.94 76.775)
+		(width 0.5)
+		(layer "B.Cu")
+		(net 6)
+	)
 	(zone
 		(net 2)
@@
 		)
 	)
-	(group ""
-		(members "07c0d147-c5f7-41c6-8d61-837e63ca47e9" "08056941-45b0-4530-b30b-e5f30cb43ee0"
-			"09f22a1b-de06-4166-ba74-86811f9893ee" "0b23b4b8-ef88-4dc0-9de0-97d78c32625e"
-			"0b7c752b-8cde-4d6f-97d3-1a923cad7c32" "0c290e95-afb1-4677-8b44-83f8416010d7"
-			"0f80edfd-90a9-4273-9899-ff4e5d15e13a" "105081dc-6b3c-4c89-b615-7ffe06b7a333"
-			"12088568-241d-4c25-abc4-505a69b1c101" "14e4bea4-f04f-4bb9-a043-2d3a47384cc4"
-			"1f574501-7a58-40a9-a87b-e08626d8fb30" "20c2cccb-d221-45cf-892b-19408d6bb29f"
-			"2453bc41-c8d1-4064-b0de-d9053af11b1c" "304bf6f6-567f-46b8-a3a8-7fc7d196b6bb"
-			"313ef089-c179-4314-b57c-2437a8066b8d" "3429bf37-6abc-485d-8c02-d750c7421474"
-			"344c3fed-35ed-444a-9955-12d594ab00c6" "40da01c3-30b4-4c16-84f9-67e8bab82545"
-			"45d664dd-2cc1-43bc-9250-6a59c314dadb" "49e9f82d-9c5c-44f9-b141-5d1ec93c588f"
-			"5642507c-2132-44d9-a8ea-96eeb222ccd0" "57bcc69b-3e11-4598-a0d4-50c96a6bda09"
-			"5deda1f3-ebbf-46b4-84d9-4a0e1931e0d2" "5f123ac7-5095-45af-ae38-d33693678013"
-			"5fecfcd0-fe33-4a8e-870b-5ca09a746edb" "652004d5-25fd-49a1-bf4c-bece1de2cc92"
-			"675375b2-0b82-4f7b-8cc0-a8537d8cd6a4" "72b7f2cd-e399-42a4-8206-cc9bd9692996"
-			"7580983d-39ff-47cc-9f3d-914a1d47828d" "75947ac4-d534-4111-a810-e17c72b76d9a"
-			"79b5bcc7-186c-4b47-8a65-f07b7fff205b" "7ef43711-9aff-4951-948e-bb7b3e59c519"
-			"8030fa2e-1c10-4884-ba70-16fb6fa7f12b" "864ea547-224f-428e-b2ab-cc75bf6bfed2"
-			"895d667a-e88e-485c-844a-5b52ccdb08f5" "899a04af-a2d8-406e-a5c0-447873c07282"
-			"8cb181ae-03e2-4e7a-89ca-59993c8bbe46" "911f9ed8-b7f9-4718-9efa-a7e43e859d04"
-			"9d5fb13a-46df-4761-8d53-6b1e6c2e418a" "a04a8bd2-b8ea-4b0b-a930-28109373e9cb"
-			"a1450ee9-de75-4f9f-87ae-7f314a1372b8" "a34d1963-c227-4645-b82d-4174d9a398e7"
-			"aa537f4c-45a9-4fd8-8b74-56fa9bb8c3a6" "abeae4b7-0345-4ed4-bfc4-0940a6fb9350"
-			"b7ee3e72-20a3-4dc0-9bed-3efe0a73e201" "b9b0a2d3-a5d1-4dc0-a933-74287f46eb21"
-			"ba1264b0-8258-4647-9368-657e30f4bf6a" "bcad0157-8792-4dab-a7a2-d4a55734b9e8"
-			"c1a4e182-caa5-415a-8974-81ec62952f72" "c3bbb92e-53f6-4c80-bbce-32964debe0bc"
-			"c6b9c619-a181-466d-94dd-d79e1f4e2e16" "cb7c5160-9867-4174-bfad-cc351df09dea"
-			"d4c1ccc0-3913-4181-8162-06400a11c6a5" "d4dcad59-270e-47bf-9322-f1425a631ce3"
-			"d7c1cd7a-1d35-4f57-aebe-6343c8811b6f" "de202138-baeb-4826-a622-4e9dd7fef2a2"
-			"e5687838-2e7e-4411-8d96-d8193874d7d8" "e951c8e2-23ad-429c-860f-f4069798c67b"
-			"ec69be76-c280-4d6b-87b3-0cf9e46fdf05" "ed5815a8-2ad1-48c9-9046-89b222ba8264"
-			"ee15ef68-f422-4dee-91e0-0163a8622be6" "ef371a5f-5c0a-4f16-936b-8c7782eb7592"
-			"fc39bdd2-eac8-4e28-b6e2-2d1c4eb03201"
-		)
-	)

Commit message: Adding git ignore
Other:
- board text added: "All units are in milimiters unles otherwiese specified"
Changed lines of the file:
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@@
 		(pad_to_mask_clearance 0)
 		(allow_soldermask_bridges_in_footprints no)
+		(aux_axis_origin 85.25 81.835)
+		(grid_origin 85.25 81.835)
 		(pcbplotparams
 			(layerselection 0x00010fc_ffffffff)
@@
 			(at 0 1.55 0)
 			(layer "F.Fab")
+			(hide yes)
 			(effects
 				(font
@@
 		)
 		(fp_text user "${REFERENCE}"
-			(at 0 -1.45 0)
+			(at 0.14 -1.455 0)
 			(layer "F.Fab")
 			(effects
@@
 			(at 0 1.5 0)
 			(layer "F.Fab")
+			(hide yes)
 			(effects
 				(font
@@
 			(at 0 1.5 0)
 			(layer "F.Fab")
+			(hide yes)
 			(effects
 				(font
@@
 			(at 0 1.5 0)
 			(layer "F.Fab")
+			(hide yes)
 			(effects
 				(font
@@
 			(at 0 3.2 0)
 			(layer "F.Fab")
+			(hide yes)
 			(effects
 				(font
@@
 			(at 0 3.2 0)
 			(layer "F.Fab")
+			(hide yes)
 			(effects
 				(font
@@
 			(at 0 1.55 0)
 			(layer "F.Fab")
+			(hide yes)
 			(effects
 				(font
@@
 		)
 		(fp_text user "${REFERENCE}"
-			(at 0 -1.45 0)
+			(at 0.16 -1.465 0)
 			(layer "F.Fab")
 			(effects
@@
 			(at 0 1.55 0)
 			(layer "F.Fab")
+			(hide yes)
 			(effects
 				(font
@@
 		)
 		(fp_text user "${REFERENCE}"
-			(at 0 -1.45 0)
+			(at 0.17 -1.47 0)
 			(layer "F.Fab")
 			(effects
@@
 			(at 0 -1.5 0)
 			(layer "B.Fab")
+			(hide yes)
 			(effects
 				(font
@@
 			(at -0.8775 -1.67 0)
 			(layer "B.Fab")
+			(hide yes)
 			(effects
 				(font
@@
 			(at 0 -2 0)
 			(layer "B.Fab")
+			(hide yes)
 			(effects
 				(font
@@
 			(at 1.12 -1.78 90)
 			(layer "B.Fab")
+			(hide yes)
 			(effects
 				(font
@@
 			(at 0 -1.5 0)
 			(layer "B.Fab")
+			(hide yes)
 			(effects
 				(font
@@
 			(at 0 -1.65 90)
 			(layer "B.Fab")
+			(hide yes)
 			(effects
 				(font
@@
 			(at 0 -1.5 0)
 			(layer "B.Fab")
+			(hide yes)
 			(effects
 				(font
@@
 			(at 0 -1.43 0)
 			(layer "B.Fab")
+			(hide yes)
 			(effects
 				(font
@@
 			(at 0 -1.17 90)
 			(layer "B.Fab")
+			(hide yes)
 			(effects
 				(font
@@
 			(at 0 -1.43 90)
 			(layer "B.Fab")
+			(hide yes)
 			(effects
 				(font
@@
 		)
 	)
+	(gr_text "All units are in milimiters unles otherwiese specified"
+		(at 64.76 92.16 0)
+		(layer "Dwgs.User")
+		(effects
+			(font
+				(size 2 2)
+				(thickness 0.3)
+			)
+			(justify left bottom)
+		)
+	)
 	(gr_text "PCB3D_BR_template"
 		(at 115.25 81.835 180)
@@
 		)
 		(height -5.04)
-		(gr_text "30.00 mm"
+		(gr_text "30.00"
 			(at 100.25 45.895 0)
 			(layer "Dwgs.User")
@@
 			(suffix "")
 			(units 3)
-			(units_format 1)
+			(units_format 0)
 			(precision 2)
 		)
@@
 		)
 		(height 3.18)
-		(gr_text "30.00 mm"
+		(gr_text "30.00"
 			(at 81.17 66.835 90)
 			(layer "Dwgs.User")
@@
 			(suffix "")
 			(units 3)
-			(units_format 1)
+			(units_format 0)
 			(precision 2)
 		)
@@
 		)
 		(height -4.68)
-		(gr_text "3.00 mm"
+		(gr_text "3.00"
 			(at 108.25 49.965 0)
 			(layer "Dwgs.User")
@@
 			(suffix "")
 			(units 3)
-			(units_format 1)
+			(units_format 0)
 			(precision 2)
 		)
@@
 		)
 		(height 4.58)
-		(gr_text "3.00 mm"
+		(gr_text "3.00"
 			(at 117.46 57.845 270)
 			(layer "Dwgs.User")
@@
 			(suffix "")
 			(units 3)
-			(units_format 1)
+			(units_format 0)
 			(precision 2)
 		)
