File: extension_template/extension_template.kicad_pcb (KiCad board)
At the start: 4 copper layers, 30 x 30 mm, 23 parts, among them IC3 TLV61225DC, J6 MISC

Commit message: Template update
Other:
- board text added: "This is needed for PCB2BLENDER plugin!"
Changed lines of the file:
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@@
 		(layer "B.SilkS")
+	)
+	(gr_line
+		(start 87.44 50.545)
+		(end 80.45 45.175)
+		(stroke
+			(width 0.2)
+			(type default)
+		)
+		(layer "Cmts.User")
 	)
 	(gr_arc
@@
 			)
 			(justify left bottom)
+		)
+	)
+	(gr_text "This is needed for PCB2BLENDER plugin!"
+		(at 55.81 44.315 0)
+		(layer "Cmts.User" knockout)
+		(effects
+			(font
+				(size 1 1)
+				(thickness 0.15)
+			)
+			(justify left bottom)
