File: extension_template/power.kicad_sch (KiCad schematic)
At the start: 5 parts, among them IC3 TLV61225DC

Commit message: Template update
Other:
- note added: "Replace with TPS61222DCKT for 2.5V>>5V"
- company: Intergalaktik d.o.o. -> ${project_creator}
- title: olimex extension template -> ${project_name} ${project_version}
- moved on the sheet: C13, C14, IC3, L2, R15

Commit message: Extension template update
Parts:
- renumbered L2 to L1
Other:
- note added: "Power Page"
- moved on the sheet: C13, C14, IC3, L1, R15

Commit message: Template update
Connections:
- net 2V5 renamed VCC_IN
- net 3V3 renamed VCC_STEP_UP
Other:
- note added: "Use TPS61222DC for 2.5V>>5V"
- note added: "Use TPS61225DC for 2.5V>>3.3V"
- note removed: "Replace with TPS61222DCKT for 2.5V>>5V"
Changed lines of the file:
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@@
+		)
+	)
+	(text "Use TPS61222DC for 2.5V>>5V"
+		(exclude_from_sim no)
+		(at 96.266 80.772 0)
+		(effects
+			(font
+				(size 1.27 1.27)
+			)
 		)
 	)
@@
 		)
 	)
-	(text "Replace with TPS61222DCKT for 2.5V>>5V"
+	(text "Use TPS61225DC for 2.5V>>3.3V"
 		(exclude_from_sim no)
 		(at 96.012 78.74 0)
@@
 		)
 	)
-	(hierarchical_label "2V5"
+	(hierarchical_label "VCC_IN"
 		(shape input)
 		(at 78.74 54.61 90)
@@
 		)
 	)
-	(hierarchical_label "3V3"
+	(hierarchical_label "VCC_STEP_UP"
 		(shape input)
 		(at 114.3 57.15 90)
