File: tmrIO/power.kicad_sch (KiCad schematic)
At the start: 5 parts, among them IC3 TLV61225DC

Commit message: Update tmrIO
Parts:
- removed L2: 4.7uH, Inductor_SMD:L_0603_1608Metric, symbol Device:L_Small
- added L1: 4.7uH, Inductor_SMD:L_0603_1608Metric, symbol Device:L_Small
Connections:
- net at IC3.5 (L): now also L1.1
- net 2V5 renamed FPGA_VCC
- net FPGA_VCC: now also L1.2
- net 3V3 renamed 5V
Other:
- note added: "Power Page"
- note added: "StepUp 2V5>>5V"
- note added: "TPS61222DC for 2.5V>>5V"
- note added: "TPS61225DC for 2.5V>>3V3"
- note removed: "StepUp 2V5>>3V3"
- company: Intergalaktik d.o.o. -> ${project_creator}
- title: olimex extension template -> ${project_name}  ${project_version} 
