File: tmrIO/main.kicad_sch (KiCad schematic)
At the start: 26 parts, among them IC1 MCP7940NT-I_SN, J6 MISC, Y1 LFXTAL016178REEL

Commit message: tmrIO update
Parts:
- added H7, H8: MountingHole, MountingHole:MountingHole_2.2mm_M2, symbol Mechanical:MountingHole
- added TP7: BAT+, TestPoint:TestPoint_Pad_D1.0mm, symbol Connector:TestPoint_Probe
- TP1: value 3V3 -> 5V
Connections:
- net +5V: now also TP1.1
- net +Exten_V: now also J6.1 (Pin_1), TP2.1
- net 2V5: now also F1.2
- net BAT+: now also TP7.1; no longer TP3.1
- net GND: now also TP3.1; no longer TP2.1
- removed net +2V5: F1.2, J6.1 (Pin_1), TP1.1
- no-connect marks 2 -> 15
Other:
- moved on the sheet: FID1, FID2, FID3, FID4, FID5, FID6, H5, H6, TP1, TP2, TP3, TP4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
