File: tmrIO/tmrIO.kicad_sch (KiCad schematic)
At the start: 6 parts, among them IC1 MCP7940NT-I_SN, J6 MISC

Commit message: Template update
Parts:
- added BT1: Battery_Cell, Battery:BatteryHolder_Keystone_2998_1x6.8mm, symbol Device:Battery_Cell
- added F1: 0805L050WR, Fuse:Fuse_0805_2012Metric, symbol Device:Fuse_Small
- added FID1, FID2, FID3, FID4, FID5, FID6: Fiducial, Fiducial:Fiducial_0.5mm_Mask1mm, symbol Mechanical:Fiducial
- added H5, H6: MountingHole, MountingHole:MountingHole_2.2mm_M2, symbol Mechanical:MountingHole
- added R1, R2, R3: 10K, Resistor_SMD:R_0402_1005Metric, symbol Device:R_Small
- added TP1: 3V3, TestPoint:TestPoint_Pad_D1.0mm, symbol Connector:TestPoint_Probe
- added TP2: 2V5, TestPoint:TestPoint_Pad_D1.0mm, symbol Connector:TestPoint_Probe
- added TP3: GND, TestPoint:TestPoint_Pad_D1.0mm, symbol Connector:TestPoint_Probe
- added TP4: MFP, TestPoint:TestPoint_Pad_D1.0mm, symbol Connector:TestPoint_Probe
- added TP5: SCL, TestPoint:TestPoint_Pad_D1.0mm, symbol Connector:TestPoint_Probe
- added TP6: SDA, TestPoint:TestPoint_Pad_D1.0mm, symbol Connector:TestPoint_Probe
- added Y1: LFXTAL016178REEL, LFXTAL016178:LFXTAL016178REEL, symbol LFXTAL016178REEL:LFXTAL016178REEL
- H3: footprint Cologne:open_cologne -> Cologne:open_cologne_small
- H4: footprint radiona:radiona -> radiona:radiona_small
- IC1: footprint MCP7940:SOIC127P600X175-8N -> MCP7940NT-I_SN:SOIC127P600X175-8N
Connections:
- net +2V5: now also F1.1, TP1.1
- net GND: now also IC1.4 (VSS), BT1.2 (-), TP2.1
- net NB_A8: now also IC1.7 (MFP), R1.2, TP4.1
- net NB_B7: now also IC1.6 (SCL), R2.2, TP5.1
- net NB_B8: now also IC1.5 (SDA), R3.2, TP6.1
- net X1: now reaches IC1.1 (X1)
- net X1: now also Y1.1 (CRYSTAL_1)
- net X2: now reaches IC1.2 (X2)
- net X2: now also Y1.4 (CRYSTAL_2)
- net BAT+: now reaches IC1.3 (VBAT)
- net BAT+: now also BT1.1 (+), TP3.1
- net 2V5: now reaches IC1.8 (VCC)
- net 2V5: now also F1.2, R1.1, R2.1, R3.1
- no-connect marks 0 -> 2
Other:
- note added: "2V5 over Resettable Fuses - PPTC 0.50A 6V 0805 >3V3"
- company: (none) -> Intergalaktik d.o.o.
- title: (none) -> olimex extension template
- moved on the sheet: H1, H2, H3, H4, J6

Commit message: Update tmrIO
Parts:
- removed BT1: Battery_Cell, Battery:BatteryHolder_Keystone_2998_1x6.8mm, symbol Device:Battery_Cell
- removed F1: 0805L050WR, Fuse:Fuse_0805_2012Metric, symbol Device:Fuse_Small
- removed FID1, FID2, FID3, FID4, FID5, FID6: Fiducial, Fiducial:Fiducial_0.5mm_Mask1mm, symbol Mechanical:Fiducial
- removed H1: Logo Intergalaktik, intergalaktik:intergalaktik, symbol Mechanical:MountingHole
- removed H2: Logo NLnet, nlnet:nlnet, symbol Mechanical:MountingHole
- removed H3: Logo OpenCologne, Cologne:open_cologne_small, symbol Mechanical:MountingHole
- removed H4: Logo Radiona, radiona:radiona_small, symbol Mechanical:MountingHole
- removed H5, H6: MountingHole, MountingHole:MountingHole_2.2mm_M2, symbol Mechanical:MountingHole
- removed IC1: MCP7940NT-I_SN, MCP7940NT-I_SN:SOIC127P600X175-8N, symbol MCP7940NT-I_SN:MCP7940NT-I_SN
- removed J6: MISC, Connector_PinSocket_2.54mm:PinSocket_2x10_P2.54mm_Vertical_SMD, symbol Connector_Generic:Conn_02x10_Odd_Even
- removed R1, R2, R3: 10K, Resistor_SMD:R_0402_1005Metric, symbol Device:R_Small
- removed TP1: 3V3, TestPoint:TestPoint_Pad_D1.0mm, symbol Connector:TestPoint_Probe
- removed TP2: 2V5, TestPoint:TestPoint_Pad_D1.0mm, symbol Connector:TestPoint_Probe
- removed TP3: GND, TestPoint:TestPoint_Pad_D1.0mm, symbol Connector:TestPoint_Probe
- removed TP4: MFP, TestPoint:TestPoint_Pad_D1.0mm, symbol Connector:TestPoint_Probe
- removed TP5: SCL, TestPoint:TestPoint_Pad_D1.0mm, symbol Connector:TestPoint_Probe
- removed TP6: SDA, TestPoint:TestPoint_Pad_D1.0mm, symbol Connector:TestPoint_Probe
- removed Y1: LFXTAL016178REEL, LFXTAL016178:LFXTAL016178REEL, symbol LFXTAL016178REEL:LFXTAL016178REEL
Connections:
- no-connect marks 2 -> 0
Other:
- added sheet Dimensions sheet (dimensions.kicad_sch)
- added sheet Main Sheet (main.kicad_sch)
- note added: "${CURRENT_DATE}"
- note added: "${project_name} ${project_version}"
- note added: "......"
- note added: "......."
- note added: "1"
- note added: "2"
- note added: "3"
- note added: "4"
- note added: "5"
- note added: "6"
- note added: "BOTTOM VIEW"
- note added: "Board Dimensions"
- note added: "CoverPage"
- note added: "First Relay"
- note added: "Index"
- note added: "MainPage"
- note added: "Page"
- note added: "PowerPage"
- note added: "Replace bottom 3D images with your PCB"
- note added: "Second Relay"
- note added: "TOP VIEW"
- note removed: "2V5 over Resettable Fuses - PPTC 0.50A 6V 0805 >3V3"
- note removed: "OLIMEX CONNECTOR"
- note removed: "POWER FLAGS"
- company: Intergalaktik d.o.o. -> ${project_creator}
- title: olimex extension template -> ${project_name}  ${project_version} 

Commit message: tmrIO update
Other:
- note removed: "Replace bottom 3D images with your PCB"
