File: tmrIO/tmrIO.kicad_pcb (KiCad board)
At the start: 4 copper layers, 26.7 x 30.5 mm, 6 parts, among them IC1 MCP7940NT-I_SN, J6 MISC

Commit message: Template update
Parts:
- added BT1: Battery_Cell, Battery:BatteryHolder_Keystone_2998_1x6.8mm, B.Cu at (103.2, 73.9)
- added F1: 0805L050WR, Fuse:Fuse_0805_2012Metric, B.Cu at (81.0, 78.8)
- added FID1: Fiducial, Fiducial:Fiducial_0.5mm_Mask1mm, F.Cu at (83.8, 60.9)
- added FID2: Fiducial, Fiducial:Fiducial_0.5mm_Mask1mm, F.Cu at (102.7, 60.9)
- added FID3: Fiducial, Fiducial:Fiducial_0.5mm_Mask1mm, F.Cu at (79.1, 89.1)
- added FID4: Fiducial, Fiducial:Fiducial_0.5mm_Mask1mm, B.Cu at (102.7, 60.9)
- added FID5: Fiducial, Fiducial:Fiducial_0.5mm_Mask1mm, B.Cu at (83.8, 60.9)
- added FID6: Fiducial, Fiducial:Fiducial_0.5mm_Mask1mm, B.Cu at (107.4, 89.1)
- added H5: MountingHole, MountingHole:MountingHole_2.2mm_M2, F.Cu at (81.2, 63.0)
- added H6: MountingHole, MountingHole:MountingHole_2.2mm_M2, F.Cu at (105.2, 63.0)
- added R1: 10K, Resistor_SMD:R_0402_1005Metric, B.Cu at (93.5, 71.3)
- added R2: 10K, Resistor_SMD:R_0402_1005Metric, B.Cu at (95.6, 71.3)
- added R3: 10K, Resistor_SMD:R_0402_1005Metric, B.Cu at (97.8, 71.3)
- added TP1: 3V3, TestPoint:TestPoint_Pad_D1.0mm, F.Cu at (81.6, 79.9)
- added TP2: 2V5, TestPoint:TestPoint_Pad_D1.0mm, F.Cu at (84.8, 79.9)
- added TP3: GND, TestPoint:TestPoint_Pad_D1.0mm, F.Cu at (103.0, 69.3)
- added TP4: MFP, TestPoint:TestPoint_Pad_D1.0mm, F.Cu at (93.5, 73.5)
- added TP5: SCL, TestPoint:TestPoint_Pad_D1.0mm, F.Cu at (96.5, 73.5)
- added TP6: SDA, TestPoint:TestPoint_Pad_D1.0mm, F.Cu at (99.5, 73.4)
- added Y1: LFXTAL016178REEL, LFXTAL016178:LFXTAL016178REEL, B.Cu at (92.8, 77.8)
- added kibuzzard-674D68C8: G***, kibuzzard-674D68C8, F.Cu at (89.0, 88.8)
- H3: footprint Cologne:open_cologne -> Cologne:open_cologne_small
- H4: footprint radiona:radiona -> radiona:radiona_small
- IC1: footprint MCP7940:SOIC127P600X175-8N -> MCP7940NT-I_SN:SOIC127P600X175-8N; moved to B.Cu
- moved IC1 64.0 mm to (90.2, 70.7)
- moved J6 58.2 mm to (93.2, 85.4)
- moved H2 46.8 mm to (83.8, 83.7)
- moved H3 31.4 mm to (101.8, 85.8)
- moved H1 28.2 mm to (88.9, 86.6)
- moved H4 25.2 mm to (92.6, 83.0)
Connections:
- IC1 pad 1: unconnected-(IC1-X1-Pad1) -> /X1
- IC1 pad 2: unconnected-(IC1-X2-Pad2) -> /X2
- IC1 pad 3: unconnected-(IC1-VBAT-Pad3) -> /BAT+
- IC1 pad 4: unconnected-(IC1-VSS-Pad4) -> GND
- IC1 pad 5: unconnected-(IC1-SDA-Pad5) -> /NB_B8
- IC1 pad 6: unconnected-(IC1-SCL-Pad6) -> /NB_B7
- IC1 pad 7: unconnected-(IC1-MFP-Pad7) -> /NB_A8
- IC1 pad 8: unconnected-(IC1-VCC-Pad8) -> /2V5
Routing:
- net /BAT+: track 0.00 -> 37.0 mm, vias 0 -> 3
- net /NB_B8: track 0.00 -> 32.3 mm, vias 0 -> 1
- net /NB_A8: track 0.00 -> 31.4 mm, vias 0 -> 1
- net /NB_B7: track 0.00 -> 27.9 mm, vias 0 -> 1
- net /2V5: track 0.00 -> 24.6 mm, vias 0 -> 4
- net GND: track 0.00 -> 15.0 mm, vias 0 -> 22
- net +2V5: track 0.00 -> 12.5 mm, vias 0 -> 1
- net /X2: track 0.00 -> 7.25 mm
- net /X1: track 0.00 -> 6.45 mm
- added copper zone on B.Cu, net GND
- added copper zone on F.Cu, net GND
- added copper zone on In1.Cu, net GND
- added copper zone on In2.Cu, net GND
Other:
- board size 26.7 x 30.5 mm -> 30 x 30 mm
- board text added: "PCB3D_BR_template"
- board text added: "PCB3D_TL_template"
- board text removed: "PCB3D_BR_tmrIO"
- board text removed: "PCB3D_TL_tmrIO"

Commit message: tmrIO update
Parts:
- added C13: 10uF, Capacitor_SMD:C_0603_1608Metric, F.Cu at (94.7, 71.4)
- added C14: 10uF, Capacitor_SMD:C_0603_1608Metric, F.Cu at (92.9, 69.1)
- added D1: SM4007, Diode_SMD:D_MELF, B.Cu at (97.6, 57.3)
- added D2: SM4007, Diode_SMD:D_MELF, B.Cu at (107.0, 57.3)
- added H7: MountingHole, MountingHole:MountingHole_2.2mm_M2, F.Cu at (90.3, 34.8)
- added H8: MountingHole, MountingHole:MountingHole_2.2mm_M2, F.Cu at (114.3, 34.8)
- added IC3: TLV61225DC, Package_TO_SOT_SMD:SOT-363_SC-70-6, F.Cu at (92.3, 71.3)
- added J1: Screw_Terminal_01x02, TerminalBlock_Phoenix:TerminalBlock_Phoenix_PT-1,5-2-3.5-H_1x02_P3.50mm_Horizontal, F.Cu at (99.6, 36.8)
- added J4: Screw_Terminal_01x02, TerminalBlock_Phoenix:TerminalBlock_Phoenix_PT-1,5-2-3.5-H_1x02_P3.50mm_Horizontal, F.Cu at (108.4, 36.8)
- added K3: G5NB-1A-HA_DC5, G5NB-1A-HA:G5NB1AHADC5, F.Cu at (99.9, 61.0)
- added K4: G5NB-1A-HA_DC5, G5NB-1A-HA:G5NB1AHADC5, F.Cu at (109.3, 61.0)
- added L1: 4.7uH, Inductor_SMD:L_0603_1608Metric, F.Cu at (92.4, 73.6)
- added Q1: MMBT3904, Package_TO_SOT_SMD:SOT-23, F.Cu at (94.5, 65.1)
- added Q2: MMBT3904, Package_TO_SOT_SMD:SOT-23, F.Cu at (101.3, 65.1)
- added R15: 10K, Resistor_SMD:R_0402_1005Metric, F.Cu at (90.1, 72.7)
- added R4: 2K, Resistor_SMD:R_0402_1005Metric, F.Cu at (91.6, 66.3)
- added R5: 2K, Resistor_SMD:R_0402_1005Metric, F.Cu at (98.4, 66.2)
- added TP7: BAT+, TestPoint:TestPoint_Pad_D1.0mm, F.Cu at (114.2, 64.7)
- TP1: value 3V3 -> 5V
- moved FID1 24.8 mm to (92.8, 37.8)
- moved FID2 24.8 mm to (111.8, 37.8)
- moved FID4 24.8 mm to (111.8, 37.8)
- moved FID5 24.8 mm to (92.8, 37.8)
- moved TP1 15.4 mm to (89.6, 66.8)
- moved FID3 9.58 mm to (88.1, 86.0)
- moved FID6 9.58 mm to (116.4, 86.0)
- moved H2 9.58 mm to (92.9, 80.5)
- moved J6 9.58 mm to (102.3, 82.2)
- moved R1 9.58 mm to (102.5, 68.2)
- moved TP4 9.58 mm to (102.5, 70.3)
- moved TP6 9.58 mm to (108.5, 70.3)
- moved kibuzzard-674D68C8 9.58 mm to (98.0, 85.6)
- moved H6 9.58 mm to (114.3, 59.8)
- moved BT1 9.58 mm to (112.2, 70.7)
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Connections:
- net /2V5 renamed /Main Sheet/2V5
- net /NB_A1 renamed /Main Sheet/NB_A1
- net /NB_A2 renamed /Main Sheet/NB_A2
- net /NB_A3 renamed /Main Sheet/NB_A3
- net /NB_A4 renamed /Main Sheet/NB_A4
- net /NB_A5 renamed /Main Sheet/NB_A5
- net /NB_A6 renamed /Main Sheet/NB_A6
- net /NB_A7 renamed /Main Sheet/NB_A7
- net /NB_A8 renamed /Main Sheet/NB_A8
- net /NB_B1 renamed /Main Sheet/NB_B1
- net /NB_B2 renamed /Main Sheet/NB_B2
- net /NB_B3 renamed /Main Sheet/NB_B3
- net /NB_B4 renamed /Main Sheet/NB_B4
- net /NB_B5 renamed /Main Sheet/NB_B5
- net /NB_B6 renamed /Main Sheet/NB_B6
- net /NB_B7 renamed /Main Sheet/NB_B7
- net /NB_B8 renamed /Main Sheet/NB_B8
- net /X1 renamed /Main Sheet/X1
- net /X2 renamed /Main Sheet/X2
- BT1 pad 1: /BAT+ -> /Main Sheet/BAT+
- F1 pad 1: +2V5 -> +Exten_V
- IC1 pad 3: /BAT+ -> /Main Sheet/BAT+
- J6 pad 1: +2V5 -> +Exten_V
- J6 pad 3: /NB_A0 -> /Main Sheet/NB_A0
- J6 pad 4: /NB_B0 -> /Main Sheet/NB_B0
- TP1 pad 1: +2V5 -> +5V
- TP2 pad 1: GND -> +Exten_V
- TP3 pad 1: /BAT+ -> GND
Routing:
- net Net-(J4-Pin_2): track 0.00 -> 60.2 mm, vias 0 -> 10
- net Net-(J1-Pin_2): track 0.00 -> 57.2 mm, vias 0 -> 10
- net /Main Sheet/BAT+: track 0.00 -> 37.5 mm, vias 0 -> 3
- net /BAT+: track 37.0 -> 0.00 mm, vias 3 -> 0
- net +5V: track 0.00 -> 36.8 mm
- net Net-(J4-Pin_1): track 0.00 -> 24.9 mm, vias 0 -> 3
- net Net-(J1-Pin_1): track 0.00 -> 23.4 mm, vias 0 -> 3
- net /Main Sheet/NB_A0: track 0.00 -> 22.7 mm, vias 0 -> 1
- net /Main Sheet/NB_B0: track 0.00 -> 15.4 mm, vias 0 -> 1
- net Net-(D2-A): track 0.00 -> 13.0 mm
- net +2V5: track 12.5 -> 0.00 mm, vias 1 -> 0
- net Net-(D1-A): track 0.00 -> 10.5 mm
- net +Exten_V: track 0.00 -> 10.2 mm, vias 0 -> 1
- net /Main Sheet/2V5: track 24.6 -> 33.7 mm, vias 4 -> 5
- net Net-(IC3-L): track 0.00 -> 3.06 mm
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Other:
- board size 30 x 30 mm -> 30 x 55 mm
- board text added: "2V5>>5V"
- board text added: "All units are in milimiters unles otherwiese specified"

Commit message: Update
Other:
- board text added: "PCB3D_BR_tmrIO"
- board text added: "PCB3D_TL_tmrIO"
- board text removed: "PCB3D_BR_template"
Changed lines of the file:
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@@
 				(type "Bottom Silk Screen")
 			)
-			(copper_finish "None")
+			(layer "F.SilkS"
+				(type "Top Silk Screen")
+			)
+			(layer "F.Paste"
+				(type "Top Solder Paste")
+			)
+			(layer "F.Mask"
+				(type "Top Solder Mask")
+				(thickness 0.01)
+			)
+			(layer "F.Cu"
+				(type "copper")
+				(thickness 0.035)
+			)
+			(layer "dielectric 1"
+				(type "prepreg")
+				(thickness 0.1)
+				(material "FR4")
+				(epsilon_r 4.5)
+				(loss_tangent 0.02)
+			)
+			(layer "In1.Cu"
+				(type "copper")
+				(thickness 0.035)
+			)
+			(layer "dielectric 2"
+				(type "core")
+				(thickness 1.24)
+				(material "FR4")
+				(epsilon_r 4.5)
+				(loss_tangent 0.02)
+			)
+			(layer "In2.Cu"
+				(type "copper")
+				(thickness 0.035)
+			)
+			(layer "dielectric 3"
+				(type "prepreg")
+				(thickness 0.1)
+				(material "FR4")
+				(epsilon_r 4.5)
+				(loss_tangent 0.02)
+			)
+			(layer "B.Cu"
+				(type "copper")
+				(thickness 0.035)
+			)
+			(layer "B.Mask"
+				(type "Bottom Solder Mask")
+				(thickness 0.01)
+			)
+			(layer "B.Paste"
+				(type "Bottom Solder Paste")
+			)
+			(layer "B.SilkS"
+				(type "Bottom Silk Screen")
+			)
+			(copper_finish "HAL SnPb")
 			(dielectric_constraints no)
 		)
 		(pad_to_mask_clearance 0)
 		(allow_soldermask_bridges_in_footprints no)
-		(aux_axis_origin 87.29 86.84)
-		(grid_origin 87.29 86.84)
+		(aux_axis_origin 85.25 81.835)
+		(grid_origin 85.25 81.835)
 		(pcbplotparams
 			(layerselection 0x00010fc_ffffffff)
@@
 		(tags "resistor")
 		(property "Reference" "R4"
-			(at -0.01 -1.03 360)
+			(at -0.01 -1.03 0)
 			(layer "F.SilkS")
 			(effects
@@
 		)
 		(property "Value" "2K"
-			(at 0 1.17 360)
+			(at 0 1.17 0)
 			(layer "F.Fab")
 			(hide yes)
@@
 		)
 		(fp_text user "${REFERENCE}"
-			(at 0 0 360)
+			(at 0 0 0)
 			(layer "F.Fab")
 			(effects
@@
 		(tags "resistor")
 		(property "Reference" "R5"
-			(at -0.02 1.02 360)
+			(at -0.02 1.02 0)
 			(layer "F.SilkS")
 			(effects
@@
 		)
 		(property "Value" "2K"
-			(at 0 1.17 360)
+			(at 0 1.17 0)
 			(layer "F.Fab")
 			(hide yes)
@@
 		)
 		(fp_text user "${REFERENCE}"
-			(at 0 0 360)
+			(at 0 0 0)
 			(layer "F.Fab")
 			(effects
@@
 		(tags "THT Terminal Block Phoenix PT-1,5-2-3.5-H pitch 3.5mm size 7x7.6mm^2 drill 1.2mm pad 2.4mm")
 		(property "Reference" "J4"
-			(at 1.76 2.37 360)
+			(at 1.76 2.37 0)
 			(layer "F.SilkS")
 			(effects
@@
 		)
 		(property "Value" "Screw_Terminal_01x02"
-			(at 1.75 5.56 360)
+			(at 1.75 5.56 0)
 			(layer "F.Fab")
 			(hide yes)
@@
 		)
 		(fp_text user "${REFERENCE}"
-			(at 1.75 2.4 360)
+			(at 1.75 2.4 0)
 			(layer "F.Fab")
 			(effects
@@
 		(tags "SOT-363 SC-70-6")
 		(property "Reference" "IC3"
-			(at -2.521361 -2.29 360)
+			(at -2.521361 -2.29 0)
 			(layer "F.SilkS")
 			(effects
@@
 		)
 		(property "Value" "TLV61225DC"
-			(at 0 2 360)
+			(at 0 2 0)
 			(layer "F.Fab")
 			(hide yes)
@@
 		(tags "THT Terminal Block Phoenix PT-1,5-2-3.5-H pitch 3.5mm size 7x7.6mm^2 drill 1.2mm pad 2.4mm")
 		(property "Reference" "J1"
-			(at 1.8 2.32 360)
+			(at 1.8 2.32 0)
 			(layer "F.SilkS")
 			(effects
@@
 		)
 		(property "Value" "Screw_Terminal_01x02"
-			(at 1.75 5.56 360)
+			(at 1.75 5.56 0)
 			(layer "F.Fab")
 			(hide yes)
@@
 		)
 		(fp_text user "${REFERENCE}"
-			(at 1.75 2.4 360)
+			(at 1.75 2.4 0)
 			(layer "F.Fab")
 			(effects
@@
 		(tags "Diode MELF ")
 		(property "Reference" "D1"
-			(at 0 2.5 360)
+			(at 0 2.5 0)
 			(layer "B.SilkS")
 			(effects
@@
 		)
 		(property "Value" "SM4007"
-			(at -0.25 -2.5 360)
+			(at -0.25 -2.5 0)
 			(layer "B.Fab")
 			(hide yes)
@@
 		)
 		(fp_text user "${REFERENCE}"
-			(at 0 2.5 360)
+			(at 0 2.5 0)
 			(layer "B.Fab")
 			(effects
@@
 		(tags "Diode MELF ")
 		(property "Reference" "D2"
-			(at 0 2.5 360)
+			(at 0 2.5 0)
 			(layer "B.SilkS")
 			(effects
@@
 		)
 		(property "Value" "SM4007"
-			(at -0.25 -2.5 360)
+			(at -0.25 -2.5 0)
 			(layer "B.Fab")
 			(hide yes)
@@
 		)
 		(fp_text user "${REFERENCE}"
-			(at 0 2.5 360)
+			(at 0 2.5 0)
 			(layer "B.Fab")
 			(effects
@@
 		)
 	)
-	(gr_text "PCB3D_BR_template"
+	(gr_text "PCB3D_TL_tmrIO"
+		(at 87.28 31.86 0)
+		(layer "Cmts.User")
+		(effects
+			(font
+				(size 0.8 0.8)
+				(thickness 0.1)
+			)
+			(justify left bottom)
+		)
+	)
+	(gr_text "PCB3D_BR_tmrIO"
 		(at 117.29 86.84 180)
 		(layer "Cmts.User")
