File: MikroBusIO/MikroBusIO.kicad_pcb (KiCad board)
At the start: 4 copper layers, 30 x 60 mm, 71 parts, among them IC1 LSF0108PWR, IC2 LSF0108PWR, IC3 TLV61225DC, J6 MISC, P1 microBus_1, P2 microBus_2, Q1 MMBT3904, Q2 MMBT3904

Commit message: Routing extensions
Parts:
- added H7: Logo MikroBus, MikroBus:mikrobus_logo, F.Cu at (99.6, 25.4)
- added H8: MountingHole, MountingHole:MountingHole_2.2mm_M2, F.Cu at (88.3, 24.9)
- added H9: MountingHole, MountingHole:MountingHole_2.2mm_M2, F.Cu at (112.2, 24.9)
- moved R3 28.6 mm to (90.5, 73.5)
- moved R4 28.3 mm to (91.7, 73.5)
- moved R5 26.9 mm to (93.0, 73.5), turned to 90 degrees
- moved R6 25.5 mm to (94.3, 73.5), turned to 90 degrees
- moved R7 24.4 mm to (95.5, 73.5), turned to 90 degrees
- moved R11 23.8 mm to (100.4, 73.5), turned to 90 degrees
- moved R8 23.4 mm to (96.7, 73.5), turned to 90 degrees
- moved R9 22.7 mm to (97.8, 73.5), turned to 90 degrees
- moved R12 22.0 mm to (101.6, 73.5), turned to 90 degrees
- moved R13 20.1 mm to (103.1, 73.5), turned to 90 degrees
- moved R14 18.8 mm to (104.1, 73.5), turned to 90 degrees
- moved R16 17.5 mm to (105.3, 73.5), turned to 90 degrees
- moved R17 16.4 mm to (106.4, 73.5), turned to 90 degrees
- moved R18 15.4 mm to (107.8, 73.2), turned to 90 degrees
- moved R19 14.7 mm to (109.2, 73.5), turned to 90 degrees
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Routing:
- net /Main Sheet/NB_A8_8P: track 0.00 -> 45.6 mm, vias 0 -> 1
- net /Main Sheet/NB_B8_8N: track 0.00 -> 32.6 mm, vias 0 -> 1
- net +VCC_LOW: track 42.6 -> 67.3 mm
- net Net-(IC2-EN): track 3.69 -> 15.3 mm
- net Net-(IC1-EN): track 3.77 -> 14.2 mm, vias 1 -> 0
- net GND: track 9.65 -> 17.1 mm, vias 6 -> 69
- net Net-(Q2-B): track 0.00 -> 1.77 mm
- net Net-(Q1-B): track 0.00 -> 1.71 mm
- net /Main Sheet/NB_B7_7N: track 14.4 -> 15.3 mm
- net /Main Sheet/NB_A7_7P: track 20.2 -> 20.9 mm
- net /Main Sheet/NB_A3_3P: track 19.3 -> 20.1 mm
- net /Main Sheet/NB_B4_4N: track 14.9 -> 15.5 mm
- net /Main Sheet/NB_A1_1P: track 20.0 -> 20.6 mm
- net /Main Sheet/NB_A4_4P: track 20.5 -> 21.1 mm
- net /Main Sheet/NB_B5_5N: track 14.4 -> 15.0 mm
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Other:
- rule pad_to_mask_clearance: 0.05 -> 0
