File: MikroBusIO/main.kicad_sch (KiCad schematic)
At the start: 65 parts, among them IC1 LSF0108PWR, IC2 LSF0108PWR, J6 MISC, P1 microBus_1, P2 microBus_2, Q1 MMBT3904, Q2 MMBT3904

Commit message: Routing extensions
Parts:
- added H7: Logo MikroBus, MikroBus:mikrobus_logo, symbol Mechanical:MountingHole
- added H8, H9: MountingHole, MountingHole:MountingHole_2.2mm_M2, symbol Mechanical:MountingHole
Other:
- moved on the sheet: FID1, FID2, FID3, FID4, FID5, FID6, H5, H6, TP1, TP2, TP3
