File: ethIO/ethIO.kicad_pcb (KiCad board)
At the start: 4 copper layers, 30 x 50 mm, 61 parts, among them IC3 TLV61225DC, J6 MISC, J7 HR911130A1, U10 RTL8211E-VB-CG, Y1 25MHz

Commit message: Updating ethIO license
Other:
- board text added: "Partial routing is taken from this repository https://github.com/rishivg/IO-SDR"
Changed lines of the file:
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@@
 	)
 	(property "project_creator" "Intergalaktik d.o.o.")
-	(property "project_license" "CERN-OHL-S v2")
+	(property "project_license" "GPL-3.0")
 	(property "project_name" "Olimex Extension ethIO")
 	(property "project_version" "v0.1")
@@
 			)
 			(justify left bottom)
+		)
+	)
+	(gr_text "Partial routing is taken from this repository\nhttps://github.com/rishivg/IO-SDR"
+		(at 53.85 23.365 0)
+		(layer "Cmts.User")
+		(effects
+			(font
+				(size 0.8 0.8)
+				(thickness 0.1)
+			)
+			(justify left bottom)
