File: ethIO/power.kicad_sch (KiCad schematic)
At the start: 5 parts, among them IC3 TLV61225DC

Commit message: Moving to v9
Changed lines of the file:
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@@
 (kicad_sch
-	(version 20231120)
+	(version 20250114)
 	(generator "eeschema")
-	(generator_version "8.0")
+	(generator_version "9.0")
 	(paper "A5")
 	(title_block
@@
 		(comment 1 "${project_license}")
 	)
+	(rectangle
+		(start 71.12 40.64)
+		(end 124.46 76.2)
+		(stroke
+			(width 0.127)
+			(type dash)
+		)
+		(fill
+			(type color)
+			(color 0 12 255 0.48)
+		)
+	)
+	(text "Up to 300-mA Output Current\n1-MHz Fixed-Frequency PWM Operation"
+		(exclude_from_sim no)
+		(at 97.79 43.434 0)
+		(effects
+			(font
+				(size 1.27 1.27)
+				(color 0 0 0 1)
+			)
+		)
+	)
+	(text "Use TPS61222DC for 2.5V>>5V"
+		(exclude_from_sim no)
+		(at 96.266 80.772 0)
+		(effects
+			(font
+				(size 1.27 1.27)
+			)
+		)
+	)
+	(text "Power Page"
+		(exclude_from_sim no)
+		(at 35.306 17.018 0)
+		(effects
+			(font
+				(size 5.08 5.08)
+				(thickness 0.762)
+				(bold yes)
+			)
+		)
+	)
+	(text "StepUp 2V5>>3V3"
+		(exclude_from_sim no)
+		(at 89.154 40.386 0)
+		(effects
+			(font
+				(size 1.27 1.27)
+				(bold yes)
+			)
+			(justify right bottom)
+		)
+	)
+	(text "Use TPS61225DC for 2.5V>>3.3V"
+		(exclude_from_sim no)
+		(at 96.012 78.74 0)
+		(effects
+			(font
+				(size 1.27 1.27)
+			)
+		)
+	)
 	(junction
 		(at 78.74 55.88)
@@
 		)
 	)
-	(rectangle
-		(start 71.12 40.64)
-		(end 124.46 76.2)
-		(stroke
-			(width 0.127)
-			(type dash)
-		)
-		(fill
-			(type color)
-			(color 0 12 255 0.48)
-		)
-	)
-	(text "Up to 300-mA Output Current\n1-MHz Fixed-Frequency PWM Operation"
-		(exclude_from_sim no)
-		(at 97.79 43.434 0)
-		(effects
-			(font
-				(size 1.27 1.27)
-				(color 0 0 0 1)
-			)
-		)
-	)
-	(text "Use TPS61222DC for 2.5V>>5V"
-		(exclude_from_sim no)
-		(at 96.266 80.772 0)
-		(effects
-			(font
-				(size 1.27 1.27)
-			)
-		)
-	)
-	(text "Power Page"
-		(exclude_from_sim no)
-		(at 35.306 17.018 0)
-		(effects
-			(font
-				(size 5.08 5.08)
-				(thickness 0.762)
-				(bold yes)
-			)
-		)
-	)
-	(text "StepUp 2V5>>3V3"
-		(exclude_from_sim no)
-		(at 89.154 40.386 0)
-		(effects
-			(font
-				(size 1.27 1.27)
-				(bold yes)
-			)
-			(justify right bottom)
-		)
-	)
-	(text "Use TPS61225DC for 2.5V>>3.3V"
-		(exclude_from_sim no)
-		(at 96.012 78.74 0)
-		(effects
-			(font
-				(size 1.27 1.27)
-			)
-		)
-	)
 	(hierarchical_label "VCC_IN"
 		(shape input)
 		(at 78.74 54.61 90)
-		(fields_autoplaced yes)
 		(effects
 			(font
@@
 		(shape input)
 		(at 114.3 57.15 90)
-		(fields_autoplaced yes)
-		(effects
-			(font
+		(effects
+			(font
