File: pwrIO/power.kicad_sch (KiCad schematic)
At the start: 5 parts, among them IC3 TLV61225DC

Commit message: PCB update
Parts:
- renumbered L2 to L1
Changed lines of the file:
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@@
 		(on_board yes)
 		(dnp no)
-		(property "Reference" "L2"
+		(property "Reference" "L1"
 			(at 96.266 51.562 90)
 			(effects
