File: dualTranslation/power.kicad_sch (KiCad schematic)
At the start: 5 parts, among them IC3 TLV61225DC

Commit message: Adding PULL UPs on LOW Level
Other:
- title: Motor driver board -> Dual Translation
Changed lines of the file:
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@@
 	(paper "A5")
 	(title_block
-		(title "Motor driver board")
-		(date "2024-11-26")
+		(title "Dual Translation")
+		(date "2024-11-29")
 		(rev "v0.1")
 		(company "Intergalaktik d.o.o.")
