File: dualTranslation/dualTranslation.kicad_pcb (KiCad board)
At the start: 4 copper layers, 39.4 x 39.2 mm, 59 parts, among them IC1 LSF0108PWR, IC2 LSF0108PWR, IC3 TLV61225DC, J1 L_dual, J2 R_dual, J6 MISC, Q1 MMBT3904, Q2 MMBT3904

Commit message: Fix #5
Connections:
- J1 pad 1: +3.3V -> +3V3
- J1 pad 2: +3.3V -> +3V3
- J2 pad 1: +3.3V -> +3V3
- J2 pad 2: +3.3V -> +3V3
Routing:
- net +3V3: track 91.9 -> 126.8 mm
- net +3.3V: track 31.6 -> 0.00 mm
- net GND: track 12.8 -> 14.4 mm
- net /NB_A8: track 42.7 -> 42.0 mm
Other:
- outline, holes or cut-outs redrawn

Commit message: V0.2 dualTranslation - it should now work
Parts:
- removed kibuzzard-6749EA83: G***, kibuzzard-6749EA83
- added kibuzzard-686100D9: G***, kibuzzard-686100D9, F.Cu at (139.9, 106.2)
